Commit message: feat: stop visualize from shadowing xacro and add host adaptors
Launch pose args stay empty so TCP and mount defaults come from xacro.
Finger travel is 0.045 m, and Franka/Marvin adaptor meshes ship with the
description.

Co-authored-by: Cursor <cursoragent@cursor.com>

File: urdf/pika_gripper.ros2_control.xacro (robot description, xacro)
@@ -4,5 +4,9 @@
   Actuated joint: ${prefix}gripper_left_joint (right finger is URDF mimic).
   use_fake_hardware:=true → mock_components/GenericSystem.
-  Limits: config/joint_limits.yaml
+  User-facing hardware params: serial_port, max_width.
+  Other safety defaults live in the plugin (see
+  pika_gripper_hardware_interface/docs/HARDWARE_PARAMETERS.md).
+  Joint travel limits: config/joint_limits.yaml (or joint_limits_file=;
+  max_width defaults to the YAML upper when left empty)
 -->
 <robot xmlns:xacro="http://www.ros.org/wiki/xacro">
@@ -13,13 +17,14 @@
       prefix:=''
       serial_port:=/dev/ttyUSB0
-      baudrate:=460800
       use_fake_hardware:=false
-      max_speed:=0.15
-      command_deadband:=0.0005
-      stale_warn_s:=0.1
-      stale_error_s:=0.5
-      activation_timeout_s:=2.0">
+      joint_limits_file:=''
+      max_width:=''">
+    <xacro:property name="limits_cfg_hw"
+      value="${xacro.load_yaml(joint_limits_file) if joint_limits_file != '' else pika_joint_limits_hw}"/>
     <xacro:property name="finger_lim"
-      value="${pika_joint_limits_hw['gripper_left_joint']['limit']}"/>
+      value="${limits_cfg_hw['gripper_left_joint']['limit']}"/>
+    <!-- Empty max_width → finger-travel upper from joint_limits YAML. -->
+    <xacro:property name="max_width_v"
+      value="${max_width if max_width != '' else finger_lim['upper']}"/>
     <ros2_control name="${name}" type="system">
       <hardware>
@@ -30,10 +35,6 @@
           <plugin>pika_gripper_hardware_interface/PikaGripperInterface</plugin>
           <param name="serial_port">${serial_port}</param>
-          <param name="baudrate">${baudrate}</param>
-          <param name="max_speed">${max_speed}</param>
-          <param name="command_deadband">${command_deadband}</param>
-          <param name="stale_warn_s">${stale_warn_s}</param>
-          <param name="stale_error_s">${stale_error_s}</param>
-          <param name="activation_timeout_s">${activation_timeout_s}</param>
+          <!-- ROS finger-travel upper clamp [m]; opening on wire ≈ 2×. -->
+          <param name="max_width">${max_width_v}</param>
         </xacro:unless>
       </hardware>

File: urdf/pika_gripper.xacro (robot description, xacro)
@@ -3,8 +3,8 @@
   Mountable AgileX Pika gripper (validated kinematics).
   Geometry: meshes/gripper_base_link.STL + meshes/pika_finray_link.STL
-  DOF: ${prefix}gripper_left_joint prismatic [0, upper]; right mimics left (×1).
+  DOF: ${prefix}gripper_left_joint prismatic [0, 0.045]; right mimics left (×1).
   Right finger mount yaw=-π; both axes local -X so +q closes toward center.
-  Limits: config/joint_limits.yaml
-  TCP / camera frames: config/gripper_tcp.yaml, config/cameras.yaml
+  Limits: config/joint_limits.yaml (or joint_limits_file= on the macro)
+  TCP / camera frames: config/gripper_tcp.yaml (or tcp_file=), config/cameras.yaml
 -->
 <robot xmlns:xacro="http://www.ros.org/wiki/xacro">
@@ -20,4 +20,6 @@
       *origin
       description_pkg:=pika_gripper_description
+      tcp_file:=''
+      joint_limits_file:=''
       tcp_xyz:=''
       tcp_rpy:=''
@@ -26,7 +28,12 @@
       d405_xyz:=''
       d405_rpy:=''">
-    <xacro:property name="finger_lim" value="${pika_joint_limits['gripper_left_joint']['limit']}"/>
-    <xacro:property name="tcp_xyz_v" value="${tcp_xyz if tcp_xyz != '' else pika_tcp['origin']['xyz']}"/>
-    <xacro:property name="tcp_rpy_v" value="${tcp_rpy if tcp_rpy != '' else pika_tcp['origin']['rpy']}"/>
+    <!-- Optional host bringup YAMLs override package defaults. -->
+    <xacro:property name="tcp_cfg"
+      value="${xacro.load_yaml(tcp_file) if tcp_file != '' else pika_tcp}"/>
+    <xacro:property name="limits_cfg"
+      value="${xacro.load_yaml(joint_limits_file) if joint_limits_file != '' else pika_joint_limits}"/>
+    <xacro:property name="finger_lim" value="${limits_cfg['gripper_left_joint']['limit']}"/>
+    <xacro:property name="tcp_xyz_v" value="${tcp_xyz if tcp_xyz != '' else tcp_cfg['origin']['xyz']}"/>
+    <xacro:property name="tcp_rpy_v" value="${tcp_rpy if tcp_rpy != '' else tcp_cfg['origin']['rpy']}"/>
     <xacro:property name="fisheye_xyz_v" value="${fisheye_xyz if fisheye_xyz != '' else pika_cameras['fisheye']['origin']['xyz']}"/>
     <xacro:property name="fisheye_rpy_v" value="${fisheye_rpy if fisheye_rpy != '' else pika_cameras['fisheye']['origin']['rpy']}"/>

File: urdf/pika_gripper_standalone.urdf.xacro (robot description, xacro)
@@ -3,4 +3,5 @@
 <robot xmlns:xacro="http://www.ros.org/wiki/xacro" name="pika_gripper_standalone">
   <xacro:arg name="serial_port" default="/dev/ttyUSB0"/>
+  <xacro:arg name="max_width" default="0.045"/>
   <xacro:arg name="use_fake_hardware" default="true"/>
   <xacro:arg name="xyz" default="0 0 0"/>
@@ -19,4 +20,5 @@
   <xacro:pika_gripper_ros2_control
     serial_port="$(arg serial_port)"
+    max_width="$(arg max_width)"
     use_fake_hardware="$(arg use_fake_hardware)"/>
 </robot>
