Commit message: fix(urdf): correct finger joint axes, symmetrize origins, add adaptor inertial

File: urdf/franka_pika_adaptor.xacro (robot description, xacro)
@@ -16,4 +16,11 @@
     </joint>
     <link name="${prefix}pika_adaptor_link">
+      <inertial>
+        <origin xyz="-0.01065 0.00003 0.00338" rpy="0 0 0"/>
+        <mass value="0.05"/>
+        <inertia
+          ixx="1.304E-05" ixy="1.072E-07" ixz="-7.348E-07"
+          iyy="3.212E-05" iyz="3.888E-09" izz="4.432E-05"/>
+      </inertial>
       <visual>
         <origin xyz="0 0 0" rpy="0 0 0"/>

File: urdf/pika_gripper.xacro (robot description, xacro)
@@ -94,8 +94,8 @@
     </link>
     <joint name="${prefix}gripper_left_joint" type="prismatic">
-      <origin xyz="0.04351 0 0.0815" rpy="0 0 0"/>
+      <origin xyz="0.03898 0 0.0815" rpy="0 0 0"/>
       <parent link="${prefix}gripper_base_link"/>
       <child link="${prefix}gripper_left_link"/>
-      <axis xyz="1 0 0"/>
+      <axis xyz="-1 0 0"/>
       <limit
         lower="${finger_lim['lower']}"
@@ -110,5 +110,5 @@
         <inertia
           ixx="3.448E-05" ixy="-4.3614E-09" ixz="-1.4473E-05"
-          iyy="3.9744E-05" iyz="-1.4956E-08" izz="1.5284E-05"/>
+          iyy="3.9744E-05" iyz="1.4911E-08" izz="1.5284E-05"/>
       </inertial>
       <visual>
@@ -117,5 +117,5 @@
           <mesh filename="package://${description_pkg}/meshes/pika_finray_link.STL"/>
         </geometry>
-        <material name="${prefix}pika_finray_gray_r">
+        <material name="${prefix}pika_finray_gray">
           <color rgba="0.75 0.75 0.78 1"/>
         </material>
@@ -129,8 +129,8 @@
     </link>
     <joint name="${prefix}gripper_right_joint" type="prismatic">
-      <origin xyz="-0.043529 0 0.0815" rpy="0 0 -3.14159"/>
+      <origin xyz="-0.03898 0 0.0815" rpy="0 0 -3.14159"/>
       <parent link="${prefix}gripper_base_link"/>
       <child link="${prefix}gripper_right_link"/>
-      <axis xyz="1 0 0"/>
+      <axis xyz="-1 0 0"/>
       <limit
         lower="${finger_lim['lower']}"
